Commit message: Add dump tranforms

File: ros/catkin_ws/src/david_conf/urdf/david.urdf (robot description, URDF)
Before this commit: robot david, 4 links, 3 joints
Links:
- added link DUL_block
- added link DUL_motor
- added link DUR_block
- added link DUR_motor
- added link map
Joints:
- added joint L_base_link_2_block_base: type fixed, parent base_link, child DUL_motor, origin xyz=0.28 0.065 0.05 rpy=0 -2.600540585471551 0, axis 1 0 0
- added joint L_dump_base_2_block: type prismatic, parent DUL_motor, child DUL_block, origin xyz=0.07 0 0 rpy=0 0 0, axis 1 0 0, limit lower=0.0 upper=0.75 effort=95 velocity=400
- added joint R_base_link_2_block_base: type fixed, parent base_link, child DUR_motor, origin xyz=0.28 -0.13 0.05 rpy=0 -2.600540585471551 0, axis 1 0 0
- added joint R_dump_base_2_block: type prismatic, parent DUR_motor, child DUR_block, origin xyz=0.07 0 0 rpy=0 0 0, axis 1 0 0, limit lower=0.0 upper=0.75 effort=95 velocity=400
- added joint maptestingjoint: type fixed, parent map, child base_link, origin xyz=0 0 0 rpy=0 0 0, axis 0 0 0
- joint loco_left: axis 0 0 0 -> 0 1 0; origin xyz=-0.34500000000000003 -0.09 0.07 rpy=0 0 0 -> xyz=-0.34500000000000003 0.27 0.07 rpy=0 0 0
- joint loco_right: axis 0 0 0 -> 0 1 0

File: ros/catkin_ws/src/david_conf/urdf/david.xacro (robot description, xacro)
@@ -10,9 +10,17 @@
   <link name="base_link" />
   <link name="laser" />
+  <!-- For testing only -->
+  <link name="map" />
+  <joint name="maptestingjoint" type="fixed">
+    <origin xyz="0 0 0" rpy = "0 0 0" />
+    <child link="base_link" />
+    <parent link="map" />
+    <axis xyz="0 0 0"/>
+  </joint>
   <!-- Dump motors -->
-  <!-- <link name="DUL_motor" /> -->
-  <!-- <link name="DUL_block" /> -->
-  <!-- <link name="DUR_motor" /> -->
-  <!-- <link name="DUR_block" /> -->
+  <link name="DUL_motor" />
+  <link name="DUL_block" />
+  <link name="DUR_motor" />
+  <link name="DUR_block" />
   <!-- <!-\- Depth motors -\-> -->
   <!-- <link name="DEL_motor" /> -->
@@ -27,4 +35,5 @@
   <!-- <link name="right_pitch_hinge" /> -->
   <!-- <link name="right_rear_pitch_pivot" /> -->
+  <!-- <link name="right_pitch_attachment" /> -->
   <!-- <link name="left_rear_pitch_pivot" /> -->
   <!-- Auger components -->
@@ -48,11 +57,38 @@
     <child link="right_loco_axle"/>
     <xacro:origin_rel xraw="-0.065" yraw="-0.09" zraw="0.07" rx="0" ry="0" rz="0" />
-    <axis xyz="0 0 0" />
+    <axis xyz="0 1 0" />
   </joint>
   <joint name="loco_left" type="continuous">
     <parent link="base_link" />
     <child link="left_loco_axle"/>
-    <xacro:origin_rel xraw="-0.065" yraw="0.09" zraw="0.07" rx="0" ry="0" rz="0" />
-    <axis xyz="0 0 0" />
+    <xacro:origin_rel xraw="-0.065" yraw="0.45" zraw="0.07" rx="0" ry="0" rz="0" />
+    <axis xyz="0 1 0" />
+  </joint>
+  <!-- Dump joints -->
+  <joint name="R_base_link_2_block_base" type="fixed">
+    <parent link="base_link" />
+    <child link="DUR_motor"/>
+    <xacro:origin_rel xraw="0.56" yraw="0.05" zraw="0.05" rx="0" ry="-2.600540585471551" rz="0" />
+    <axis xyz="1 0 0" />
+  </joint>
+  <joint name="R_dump_base_2_block" type="prismatic">
+    <limit lower="0.0" upper="0.75" effort="95" velocity="400" />
+    <parent link="DUR_motor" />
+    <child link="DUR_block"/>
+    <origin xyz="0.07 0 0" rpy="0 0 0"/>
+    <axis xyz="1 0 0" />
+  </joint>
+  <joint name="L_base_link_2_block_base" type="fixed">
+    <parent link="base_link" />
+    <child link="DUL_motor"/>
+    <xacro:origin_rel xraw="0.56" yraw="${0.05 + 0.195}" zraw="0.05" rx="0" ry="-2.600540585471551" rz="0" />
+    <axis xyz="1 0 0" />
+  </joint>
+  <joint name="L_dump_base_2_block" type="prismatic">
+    <limit lower="0.0" upper="0.75" effort="95" velocity="400" />
+    <parent link="DUL_motor" />
+    <child link="DUL_block"/>
+    <origin xyz="0.07 0 0" rpy="0 0 0"/>
+    <axis xyz="1 0 0" />
   </joint>
 </robot>

Commit message: Emergency commit

File: ros/catkin_ws/src/david_conf/urdf/david.urdf (robot description, URDF)
Before this commit: robot david, 9 links, 8 joints
Links:
- added link right_pitch_attachment
- added link right_pitch_hinge
- added link right_rear_pitch_pivot
Joints:
- added joint R_base_2_front_hinge: type revolute, parent base_link, child right_pitch_hinge, origin xyz=0.33499999999999996 -0.19999999999999998 0.165 rpy=0 0 0, axis 0 1 0, limit lower=0.0 upper=0.75 effort=95 velocity=400
- added joint R_base_2_rear_pivot: type fixed, parent base_link, child right_rear_pitch_pivot, origin xyz=-0.38 -0.19999999999999998 0.28 rpy=0 0 0, axis 0 0 0
- added joint R_hinge_2_attachment: type fixed, parent right_pitch_hinge, child right_pitch_attachment, origin xyz=0.38 0 0 rpy=0 0 0, axis 0 1 0
- joint L_base_link_2_block_base: origin xyz=0.28 0.065 0.05 rpy=0 -2.600540585471551 0 -> xyz=0.28 0.135 0.05 rpy=0 -2.600540585471551 0

File: ros/catkin_ws/src/david_conf/urdf/david.xacro (robot description, xacro)
@@ -33,8 +33,9 @@
   <xacro:property name="pitch_pivot_attachment_length" value="0.37" />
   <!-- <link name="left_pitch_hinge" /> -->
-  <!-- <link name="right_pitch_hinge" /> -->
-  <!-- <link name="right_rear_pitch_pivot" /> -->
-  <!-- <link name="right_pitch_attachment" /> -->
   <!-- <link name="left_rear_pitch_pivot" /> -->
+  <!-- <link nameright="left_pitch_attachment" /> -->
+  <link name="right_pitch_hinge" />
+  <link name="right_rear_pitch_pivot" />
+  <link name="right_pitch_attachment" />
   <!-- Auger components -->
   <xacro:property name="auger_length" value="0.71" />
@@ -82,5 +83,5 @@
     <parent link="base_link" />
     <child link="DUL_motor"/>
-    <xacro:origin_rel xraw="0.56" yraw="${0.05 + 0.195}" zraw="0.05" rx="0" ry="-2.600540585471551" rz="0" />
+    <xacro:origin_rel xraw="0.56" yraw="${0.05 + 0.265}" zraw="0.05" rx="0" ry="-2.600540585471551" rz="0" />
     <axis xyz="1 0 0" />
   </joint>
@@ -92,3 +93,23 @@
     <axis xyz="1 0 0" />
   </joint>
+  <!-- Pitch links -->
+  <joint name="R_base_2_rear_pivot" type="fixed">
+    <parent link="base_link" />
+    <child link="right_rear_pitch_pivot"/>
+    <xacro:origin_rel xraw="-0.10" yraw="-0.02" zraw="0.28" rx="0" ry="0" rz="0" />
+    <axis xyz="0 0 0" />
+  </joint>
+  <joint name="R_base_2_front_hinge" type="revolute">
+    <limit lower="0.0" upper="0.75" effort="95" velocity="400" />
+    <parent link="base_link" />
+    <child link="right_pitch_hinge"/>
+    <xacro:origin_rel xraw="0.615" yraw="-0.02" zraw="0.165" rx="0" ry="0" rz="0" />
+    <axis xyz="0 1 0" />
+  </joint>
+  <joint name="R_hinge_2_attachment" type="fixed">
+    <parent link="right_pitch_hinge" />
+    <child link="right_pitch_attachment"/>
+    <origin xyz="0.38 0 0"  rpy="0 0 0" />
+    <axis xyz="0 1 0" />
+  </joint>
 </robot>

Commit message: Add pitch assembly

File: ros/catkin_ws/src/david_conf/urdf/david.urdf (robot description, URDF)
Before this commit: robot david, 12 links, 11 joints
Links:
- added link DER_block
- added link DER_motor
- added link auger_hole
- added link auger_tip
Joints:
- added joint R_DER_block_2_auger_hole: type fixed, parent DER_block, child auger_hole, origin xyz=0.09 0.11 0 rpy=0 0 0, axis 0 0 0
- added joint R_DER_motor_2_DER_block: type prismatic, parent DER_motor, child DER_block, origin xyz=0.07 0 0 rpy=0 0 0, axis 1 0 0, limit lower=0.0 upper=0.48 effort=95 velocity=400
- added joint R_auger_hole_2_auger_tip: type fixed, parent auger_hole, child auger_tip, origin xyz=-0.71 0 0 rpy=0 0 0, axis 0 0 0
- added joint R_hinge_2_DEL_motor: type fixed, parent right_pitch_hinge, child DER_motor, origin xyz=0 0.085 0 rpy=0 0 0, axis 0 0 0
- joint R_base_2_front_hinge: limit lower=0.0 upper=0.75 effort=95 velocity=400 -> lower=-2.600540585471551 upper=-1.7126933813990604 effort=95 velocity=400

File: ros/catkin_ws/src/david_conf/urdf/david.xacro (robot description, xacro)
@@ -26,6 +26,6 @@
   <!-- <link name="DEL_motor" /> -->
   <!-- <link name="DEL_block" /> -->
-  <!-- <link name="DER_motor" /> -->
-  <!-- <link name="DER_block" /> -->
+  <link name="DER_motor" />
+  <link name="DER_block" />
   <!-- Pitch components -->
   <xacro:property name="pitch_pivot_attachment_length" value="0.37" />
@@ -40,7 +40,6 @@
   <!-- Auger components -->
   <xacro:property name="auger_length" value="0.71" />
-  <!-- <link name="depth_motor_axle" /> -->
-  <!-- <link name="auger_tip" /> -->
-  <!-- <link name="auger_hole"/> -->
+  <link name="auger_tip" />
+  <link name="auger_hole"/>
   <!-- Locomotion component -->
   <link name="left_loco_axle" />
@@ -100,6 +99,8 @@
     <axis xyz="0 0 0" />
   </joint>
+  <xacro:property name="hinge_max" value="-1.7126933813990604" />
+  <xacro:property name="hinge_min" value="-2.600540585471551" />
   <joint name="R_base_2_front_hinge" type="revolute">
-    <limit lower="0.0" upper="0.75" effort="95" velocity="400" />
+    <limit lower="${hinge_min}" upper="${hinge_max}" effort="95" velocity="400" />
     <parent link="base_link" />
     <child link="right_pitch_hinge"/>
@@ -113,3 +114,30 @@
     <axis xyz="0 1 0" />
   </joint>
+  <!-- Depth joints -->
+  <joint name="R_hinge_2_DEL_motor" type="fixed" >
+    <parent link="right_pitch_hinge" />
+    <child link="DER_motor"/>
+    <origin xyz="0 0.085 0"  rpy="0 0 0" />
+    <axis xyz="0 0 0" />
+  </joint>
+  <joint name="R_DER_motor_2_DER_block" type="prismatic" >
+    <limit lower="0.0" upper="0.48" effort="95" velocity="400" />
+    <parent link="DER_motor" />
+    <child link="DER_block"/>
+    <origin xyz="0.07 0 0" rpy="0 0 0"/>
+    <axis xyz="1 0 0" />
+  </joint>
+  <!-- Auger joints -->
+  <joint name="R_DER_block_2_auger_hole" type="fixed" >
+    <parent link="DER_block" />
+    <child link="auger_hole"/>
+    <origin xyz="0.09 0.11 0"  rpy="0 0 0" />
+    <axis xyz="0 0 0" />
+  </joint>
+  <joint name="R_auger_hole_2_auger_tip" type="fixed" >
+    <parent link="auger_hole" />
+    <child link="auger_tip"/>
+    <origin xyz="-0.71 0 0"  rpy="0 0 0" />
+    <axis xyz="0 0 0" />
+  </joint>
 </robot>

Commit message: Improve joint naming convention

File: ros/catkin_ws/src/david_conf/urdf/david.urdf (robot description, URDF)
Before this commit: robot david, 16 links, 15 joints
Joints:
- removed joint L_dump_base_2_block
- removed joint R_DER_block_2_auger_hole
- removed joint R_DER_motor_2_DER_block
- removed joint R_base_2_front_hinge
- removed joint R_dump_base_2_block
- added joint auger_rotation: type continuous, parent DER_block, child auger_hole, origin xyz=0.09 0.11 0 rpy=0 0 0, axis 1 0 0, limit effort=0.95 velocity=4000
- added joint depth: type prismatic, parent DER_motor, child DER_block, origin xyz=0.07 0 0 rpy=0 0 0, axis 1 0 0, limit lower=0.0 upper=0.48 effort=95 velocity=400
- added joint left_dump: type prismatic, parent DUL_motor, child DUL_block, origin xyz=0.07 0 0 rpy=0 0 0, axis 1 0 0, limit lower=0.0 upper=0.75 effort=95 velocity=400
- added joint pitch: type revolute, parent base_link, child right_pitch_hinge, origin xyz=0.33499999999999996 -0.19999999999999998 0.165 rpy=0 0 0, axis 0 1 0, limit lower=-2.600540585471551 upper=-1.7126933813990604 effort=95 velocity=400
- added joint right_dump: type prismatic, parent DUR_motor, child DUR_block, origin xyz=0.07 0 0 rpy=0 0 0, axis 1 0 0, limit lower=0.0 upper=0.75 effort=95 velocity=400
- joint loco_left: limit (none) -> effort=0.95 velocity=1000
- joint loco_right: limit (none) -> effort=0.95 velocity=1000

File: ros/catkin_ws/src/david_conf/urdf/david.xacro (robot description, xacro)
@@ -54,4 +54,5 @@
   <!-- Locomotion joints -->
   <joint name="loco_right" type="continuous">
+    <limit effort="0.95" velocity="1000" />
     <parent link="base_link" />
     <child link="right_loco_axle"/>
@@ -60,4 +61,5 @@
   </joint>
   <joint name="loco_left" type="continuous">
+    <limit effort="0.95" velocity="1000" />
     <parent link="base_link" />
     <child link="left_loco_axle"/>
@@ -72,5 +74,5 @@
     <axis xyz="1 0 0" />
   </joint>
-  <joint name="R_dump_base_2_block" type="prismatic">
+  <joint name="right_dump" type="prismatic">
     <limit lower="0.0" upper="0.75" effort="95" velocity="400" />
     <parent link="DUR_motor" />
@@ -85,5 +87,5 @@
     <axis xyz="1 0 0" />
   </joint>
-  <joint name="L_dump_base_2_block" type="prismatic">
+  <joint name="left_dump" type="prismatic">
     <limit lower="0.0" upper="0.75" effort="95" velocity="400" />
     <parent link="DUL_motor" />
@@ -101,5 +103,5 @@
   <xacro:property name="hinge_max" value="-1.7126933813990604" />
   <xacro:property name="hinge_min" value="-2.600540585471551" />
-  <joint name="R_base_2_front_hinge" type="revolute">
+  <joint name="pitch" type="revolute">
     <limit lower="${hinge_min}" upper="${hinge_max}" effort="95" velocity="400" />
     <parent link="base_link" />
@@ -121,5 +123,5 @@
     <axis xyz="0 0 0" />
   </joint>
-  <joint name="R_DER_motor_2_DER_block" type="prismatic" >
+  <joint name="depth" type="prismatic" >
     <limit lower="0.0" upper="0.48" effort="95" velocity="400" />
     <parent link="DER_motor" />
@@ -129,9 +131,10 @@
   </joint>
   <!-- Auger joints -->
-  <joint name="R_DER_block_2_auger_hole" type="fixed" >
+  <joint name="auger_rotation" type="continuous" >
+    <limit effort="0.95" velocity="4000" />
     <parent link="DER_block" />
     <child link="auger_hole"/>
     <origin xyz="0.09 0.11 0"  rpy="0 0 0" />
-    <axis xyz="0 0 0" />
+    <axis xyz="1 0 0" />
   </joint>
   <joint name="R_auger_hole_2_auger_tip" type="fixed" >

Commit message: Update urdfs

File: ros/catkin_ws/src/david_conf/urdf/david.urdf (robot description, URDF)
Before this commit: robot david, 16 links, 15 joints
Links:
- added link left_pitch_hinge
Joints:
- removed joint pitch
- added joint L_pitch: type revolute, parent base_link, child left_pitch_hinge, origin xyz=0.33499999999999996 0.18 0.165 rpy=0 0 0, axis 0 1 0, limit lower=-2.600540585471551 upper=-1.7126933813990604 effort=95 velocity=400, mimic joint=R_pitch
- added joint R_pitch: type revolute, parent base_link, child right_pitch_hinge, origin xyz=0.33499999999999996 -0.19999999999999998 0.165 rpy=0 0 0, axis 0 1 0, limit lower=-2.600540585471551 upper=-1.7126933813990604 effort=95 velocity=400
- joint auger_rotation: origin xyz=0.09 0.11 0 rpy=0 0 0 -> xyz=-0.11 0.11 0 rpy=0 0 0

File: ros/catkin_ws/src/david_conf/urdf/david.xacro (robot description, xacro)
@@ -32,5 +32,5 @@
   <xacro:property name="min_pitch_length" value="0.36" />
   <xacro:property name="pitch_pivot_attachment_length" value="0.37" />
-  <!-- <link name="left_pitch_hinge" /> -->
+  <link name="left_pitch_hinge" />
   <!-- <link name="left_rear_pitch_pivot" /> -->
   <!-- <link nameright="left_pitch_attachment" /> -->
@@ -103,9 +103,18 @@
   <xacro:property name="hinge_max" value="-1.7126933813990604" />
   <xacro:property name="hinge_min" value="-2.600540585471551" />
-  <joint name="pitch" type="revolute">
+  <joint name="R_pitch" type="revolute">
     <limit lower="${hinge_min}" upper="${hinge_max}" effort="95" velocity="400" />
     <parent link="base_link" />
     <child link="right_pitch_hinge"/>
     <xacro:origin_rel xraw="0.615" yraw="-0.02" zraw="0.165" rx="0" ry="0" rz="0" />
+    <axis xyz="0 1 0" />
+  </joint>
+  <!-- If you change the pitch lengths please adjust the action server as well -->
+  <joint name="L_pitch" type="revolute">
+    <mimic joint="R_pitch" />
+    <limit lower="${hinge_min}" upper="${hinge_max}" effort="95" velocity="400" />
+    <parent link="base_link" />
+    <child link="left_pitch_hinge"/>
+    <xacro:origin_rel xraw="0.615" yraw="0.36" zraw="0.165" rx="0" ry="0" rz="0" />
     <axis xyz="0 1 0" />
   </joint>
@@ -135,5 +144,5 @@
     <parent link="DER_block" />
     <child link="auger_hole"/>
-    <origin xyz="0.09 0.11 0"  rpy="0 0 0" />
+    <origin xyz="-0.11 0.11 0"  rpy="0 0 0" />
     <axis xyz="1 0 0" />
   </joint>

Commit message: Update urdf

File: ros/catkin_ws/src/david_conf/urdf/david.urdf (robot description, URDF)
Before this commit: robot david, 17 links, 16 joints
Links:
- added link DEL_block
- added link DEL_motor
Joints:
- removed joint R_hinge_2_DEL_motor
- removed joint depth
- added joint L_depth: type prismatic, parent DEL_motor, child DEL_block, origin xyz=0.07 0 0 rpy=0 0 0, axis 1 0 0, limit lower=0.0 upper=0.48 effort=95 velocity=400
- added joint L_hinge_2_DEL_motor: type fixed, parent left_pitch_hinge, child DEL_motor, origin xyz=0 -0.085 0 rpy=0 0 0, axis 0 0 0
- added joint R_depth: type prismatic, parent DER_motor, child DER_block, origin xyz=0.07 0 0 rpy=0 0 0, axis 1 0 0, limit lower=0.0 upper=0.48 effort=95 velocity=400
- added joint R_hinge_2_DER_motor: type fixed, parent right_pitch_hinge, child DER_motor, origin xyz=0 0.085 0 rpy=0 0 0, axis 0 0 0

File: ros/catkin_ws/src/david_conf/urdf/david.xacro (robot description, xacro)
@@ -24,6 +24,6 @@
   <link name="DUR_block" />
   <!-- <!-\- Depth motors -\-> -->
-  <!-- <link name="DEL_motor" /> -->
-  <!-- <link name="DEL_block" /> -->
+  <link name="DEL_motor" />
+  <link name="DEL_block" />
   <link name="DER_motor" />
   <link name="DER_block" />
@@ -34,5 +34,5 @@
   <link name="left_pitch_hinge" />
   <!-- <link name="left_rear_pitch_pivot" /> -->
-  <!-- <link nameright="left_pitch_attachment" /> -->
+ <!-- <link nameright="left_pitch_attachment" /> -->
   <link name="right_pitch_hinge" />
   <link name="right_rear_pitch_pivot" />
@@ -119,4 +119,17 @@
     <axis xyz="0 1 0" />
   </joint>
+  <joint name="L_hinge_2_DEL_motor" type="fixed" >
+    <parent link="left_pitch_hinge" />
+    <child link="DEL_motor"/>
+    <origin xyz="0 -0.085 0"  rpy="0 0 0" />
+    <axis xyz="0 0 0" />
+  </joint>
+  <joint name="L_depth" type="prismatic" >
+    <limit lower="0.0" upper="0.48" effort="95" velocity="400" />
+    <parent link="DEL_motor" />
+    <child link="DEL_block"/>
+    <origin xyz="0.07 0 0" rpy="0 0 0"/>
+    <axis xyz="1 0 0" />
+  </joint>
   <joint name="R_hinge_2_attachment" type="fixed">
     <parent link="right_pitch_hinge" />
@@ -126,5 +139,5 @@
   </joint>
   <!-- Depth joints -->
-  <joint name="R_hinge_2_DEL_motor" type="fixed" >
+  <joint name="R_hinge_2_DER_motor" type="fixed" >
     <parent link="right_pitch_hinge" />
     <child link="DER_motor"/>
@@ -132,5 +145,5 @@
     <axis xyz="0 0 0" />
   </joint>
-  <joint name="depth" type="prismatic" >
+  <joint name="R_depth" type="prismatic" >
     <limit lower="0.0" upper="0.48" effort="95" velocity="400" />
     <parent link="DER_motor" />

Commit message: Update urdf

File: ros/catkin_ws/src/david_conf/urdf/david.urdf (robot description, URDF)
Before this commit: robot david, 19 links, 18 joints
Joints:
- joint base2laser: origin xyz=0 0 0 rpy=0 0 0 -> xyz=-0.325 -0.0050000000000000044 0.025 rpy=0 0 3.14159

File: ros/catkin_ws/src/david_conf/urdf/david.xacro (robot description, xacro)
@@ -47,9 +47,10 @@
   <!-- Joints -->
   <joint name="base2laser" type="fixed">
-    <origin xyz="0 0 0" rpy="0 0 0" />
+    <xacro:origin_rel xraw="-0.045" yraw="0.175" zraw="0.025" rx="0" ry="0" rz="3.14159" />
     <parent link="base_link" />
     <child link="laser" />
     <axis xyz="0 0 0"/>
   </joint>
+  <!-- 2.5 up 4.5 -x 17.5 y -->
   <!-- Locomotion joints -->
   <joint name="loco_right" type="continuous">

Commit message: Scripting and xacro updates

File: ros/catkin_ws/src/david_conf/urdf/david.urdf (robot description, URDF)
Before this commit: robot david, 19 links, 18 joints
Joints:
- joint base2laser: origin xyz=-0.325 -0.0050000000000000044 0.025 rpy=0 0 3.14159 -> xyz=-0.325 -0.0050000000000000044 0.025 rpy=0 0 0

File: ros/catkin_ws/src/david_conf/urdf/david.xacro (robot description, xacro)
@@ -47,5 +47,5 @@
   <!-- Joints -->
   <joint name="base2laser" type="fixed">
-    <xacro:origin_rel xraw="-0.045" yraw="0.175" zraw="0.025" rx="0" ry="0" rz="3.14159" />
+    <xacro:origin_rel xraw="-0.045" yraw="0.175" zraw="0.025" rx="0" ry="0" rz="0" />
     <parent link="base_link" />
     <child link="laser" />
